File: PCB/Shinonome.kicad_pcb (KiCad board)
At the start: 2 copper layers, 41 parts, among them J1 MJ-4PP-9, SW1 SW_PUSH, SW10 SW_PUSH, SW11 SW_PUSH, SW12 SW_PUSH, SW13 SW_PUSH, SW14 SW_PUSH, SW15 SW_PUSH, SW16 SW_PUSH, SW17 SW_PUSH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

Commit message: first pass pcb complete
Parts:
- added G***: LOGO, Shinonome:kanji, F.Cu at (145.7, 107.6)
- added Ref**: Val**, kbd:HOLE, F.Cu at (187.8, 76.5)
- added Ref**: Val**, kbd:HOLE, F.Cu at (92.8, 85.9)
- added Ref**: Val**, kbd:HOLE, F.Cu at (92.8, 143.5)
- added Ref**: Val**, kbd:HOLE, F.Cu at (187.8, 153.2)
- added Ref**: Val**, kbd:HOLE, F.Cu at (198.0, 122.1)
- added U2: ProMicro, kbd:ProMicro_v2_Backside, F.Cu at (121.8, 86.9)
- SW1, SW10, SW11, SW12, SW13, SW14, SW15, SW16, SW17, SW18, SW19, SW2, SW3, SW4, SW5, SW6, SW7, SW8, SW9: footprint kbd:CherryMX_Hotswap -> helix:MX_ALPS_PG1350_noLed
- U1: footprint kbd:ProMicro_v2 -> kbd:ProMicro_v2_Backside; moved to B.Cu
- moved D19 170.3 mm to (198.0, 141.9)
- moved D18 157.7 mm to (198.0, 118.2)
- moved D17 153.8 mm to (179.0, 151.4)
- moved SW16 145.5 mm to (179.0, 124.4)
- moved SW17 141.3 mm to (179.0, 143.5)
- moved D16 140.6 mm to (179.0, 132.4)
- moved D15 129.5 mm to (179.0, 113.4)
- moved SW15 126.6 mm to (179.0, 105.4)
- moved D14 120.6 mm to (179.0, 94.3)
- moved SW13 119.9 mm to (159.9, 143.5)
- moved D13 119.1 mm to (159.9, 151.4)
- moved SW12 108.2 mm to (159.9, 124.4)
- moved SW14 108.2 mm to (179.0, 86.3)
- moved D12 104.5 mm to (159.9, 132.4)
- moved D10 92.8 mm to (159.9, 94.3)
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Routing:
- net col4: track 0.00 -> 202.0 mm, vias 0 -> 3
- net col3: track 0.00 -> 188.5 mm, vias 0 -> 1
- net row2: track 0.00 -> 174.4 mm, vias 0 -> 1
- net col5: track 0.00 -> 168.6 mm, vias 0 -> 5
- net col0: track 0.00 -> 151.7 mm, vias 0 -> 5
- net GND: track 0.00 -> 151.3 mm
- net reset: track 0.00 -> 145.6 mm, vias 0 -> 2
- net col1: track 0.00 -> 140.2 mm, vias 0 -> 1
- net VCC: track 0.00 -> 137.0 mm, vias 0 -> 4
- net row1: track 0.00 -> 128.5 mm
- net row3: track 0.00 -> 127.8 mm, vias 0 -> 2
- net col2: track 0.00 -> 123.4 mm
- net row0: track 0.00 -> 116.8 mm
- net data: track 0.00 -> 110.2 mm, vias 0 -> 1
- net Net-(D1-Pad2): track 0.00 -> 20.6 mm
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- added copper zone on B.Cu, net GND
- added copper zone on F.Cu, net GND
Other:
- board outline added: 127.7 x 87.9 mm
- board text added: "Shinonome PCB by @SA_EndlessGame"

Commit message: added logos and removed confusing warning from PM footprint
Parts:
- removed Ref** (x5): Val**, kbd:HOLE
- added G***: LOGO, Shinonome:emptystringLogo, B.Cu at (135.2, 111.6)
- moved G*** 1.44 mm to (147.2, 107.4)
Other:
- board text added: "Shinonome by emptystring @SA_EndlessGame"
- board text removed: "Shinonome PCB by @SA_EndlessGame"
